Commit message: MApping fixed

File: src/drone_bringup/models/x500_vision_lidar/model.urdf.xacro (robot description, xacro)
@@ -24,10 +24,10 @@
     <origin xyz="0 0 0.12" rpy="0 0 0"/>
   </joint>
-  <!-- ═══ Camera: 15cm forward, 5cm below, pitched 15° down ═══ -->
+  <!-- ═══ Camera: 15cm forward, 5cm below, pitched 25° down ═══ -->
   <link name="camera_link"/>
   <joint name="camera_joint" type="fixed">
     <parent link="base_link"/>
     <child link="camera_link"/>
-    <origin xyz="0.15 0 -0.05" rpy="0 0.26 0"/>
+    <origin xyz="0.15 0 -0.05" rpy="0 0.44 0"/>
   </joint>
   <!-- Optical frame: converts URDF convention → OpenCV convention.
